Commit message: Add other things

File: src/robot_package/urdf/rover/rover_manipulator_only.xacro (robot description, xacro)
@@ -1,9 +1,3 @@
-<robot xmlns:xacro="http://www.ros.org/wiki/xacro" name="robot_name">
-    <link name="base_link" />
+<robot xmlns:xacro="http://www.ros.org/wiki/xacro" name="robot">
     <xacro:include filename="$(find robot_package)/urdf/rover_manipulator/rover_manipulator.xacro"/>
-    <joint name="base_link_to_manipulator_link_joint" type="fixed">
-        <origin xyz="0 0 0" rpy="0 0 ${PI}"/>
-        <parent link="base_link"/>
-        <child link="manipulator_link"/>
-    </joint>
 </robot>

File: src/robot_package/urdf/rover_manipulator/rover_manipulator.xacro (robot description, xacro)
@@ -5,18 +5,19 @@
   <xacro:include filename="$(find robot_package)/urdf/rover_manipulator/utils/macros.xacro" />
   <xacro:property name="PI" value="3.1415926535897931"/>
-  <xacro:property name="mass" value="1" />
+  <xacro:property name="mass" value="0.01" />
   <xacro:property name="width" value="1"/>
   <xacro:property name="height" value="1" />
-  <!-- New dummy root link -->
-  <link name="dummy_root_link">
-    <inertial>
-      <mass value="0.0"/>
-      <origin xyz="0 0 0" rpy="0 0 0"/>
-  </link>
-  <!-- Fixed joint connecting dummy root to original root -->
-  <joint name="fixed_joint" type="fixed">
-    <parent link="dummy_root_link"/>
+  <gazebo>
+      <plugin filename="libgazebo_ros_control.so" name="gazebo_ros_control">
+        <robotNamespace>/robot</robotNamespace>
+        <robotSimType>gazebo_ros_control/DefaultRobotHWSim</robotSimType>
+      </plugin>
+  </gazebo>
+  <link name="base_link" />
+  <joint name="base_link_to_manipulator_link_joint" type="fixed">
+    <origin xyz="0 0 0" rpy="0 0 ${-PI}"/>
+    <parent link="base_link"/>
+    <kinematic>true</kinematic>
     <child link="manipulator_link"/>
-    <origin xyz="0 0 0" rpy="0 0 0"/>
   </joint>
   <link name="manipulator_link">
@@ -114,6 +115,6 @@
     <inertial>
       <origin xyz="0 0 0" rpy="0 0 0"/>
-      <mass value="${mass}"/>
-      <xacro:box_inertia mass="${mass}" width="${width}" height="${height}" />
+      <mass value="0.01"/>
+      <xacro:box_inertia mass="0.01" width="${width}" height="${height}" />
     </inertial>
   </link>
@@ -128,6 +129,6 @@
     <inertial>
       <origin xyz="0 0 0" rpy="0 0 0"/>
-      <mass value="${mass}"/>
-      <xacro:box_inertia mass="${mass}" width="${width}" height="${height}" />
+      <mass value="0.01"/>
+      <xacro:box_inertia mass="0.01" width="${width}" height="${height}" />
     </inertial>
   </link>
@@ -142,6 +143,6 @@
     <inertial>
       <origin xyz="0 0 0" rpy="0 0 0"/>
-      <mass value="${mass}"/>
-      <xacro:box_inertia mass="${mass}" width="${width}" height="${height}" />
+      <mass value="0.01"/>
+      <xacro:box_inertia mass="0.01" width="${width}" height="${height}" />
     </inertial>
   </link>
@@ -156,6 +157,6 @@
     <inertial>
       <origin xyz="0 0 0" rpy="0 0 0"/>
-      <mass value="${mass}"/>
-      <xacro:box_inertia mass="${mass}" width="${width}" height="${height}" />
+      <mass value="0.01"/>
+      <xacro:box_inertia mass="0.01" width="${width}" height="${height}" />
     </inertial>
   </link>
@@ -170,6 +171,6 @@
     <inertial>
       <origin xyz="0 0 0" rpy="0 0 0"/>
-      <mass value="${mass}"/>
-      <xacro:box_inertia mass="${mass}" width="${width}" height="${height}" />
+      <mass value="0.01"/>
+      <xacro:box_inertia mass="0.01" width="${width}" height="${height}" />
     </inertial>
   </link>
@@ -184,9 +185,9 @@
     <inertial>
       <origin xyz="0 0 0" rpy="0 0 0"/>
-      <mass value="${mass}"/>
-      <xacro:box_inertia mass="${mass}" width="${width}" height="${height}" />
-    </inertial>
-  </link>
-  <joint name="joint0" type="revolute">
+      <mass value="0.01"/>
+      <xacro:box_inertia mass="0.01" width="${width}" height="${height}" />
+    </inertial>
+  </link>
+  <joint name="joint1" type="revolute">
     <origin xyz="0 0 0" rpy="0 0 0"/>
     <parent link="manipulator_link"/>
@@ -196,5 +197,5 @@
     <dynamics damping="0.7"/>
   </joint>
-  <joint name="joint1" type="revolute">
+  <joint name="joint2" type="revolute">
     <origin xyz="0.0015 0 0.09" rpy="0 0 0"/>
     <parent link="shoulder_pan_link"/>
@@ -204,5 +205,5 @@
     <dynamics damping="0.7"/>
   </joint>
-  <joint name="joint2" type="revolute">
+  <joint name="joint3" type="revolute">
     <origin xyz="-0.00131 0 0.52453" rpy="${PI / 2} 0 0"/>
     <parent link="shoulder_tilt_link"/>
@@ -213,5 +214,5 @@
     <dynamics damping="0.7"/>
   </joint>
-  <joint name="joint3" type="revolute">
+  <joint name="joint4" type="revolute">
     <origin xyz="0.00019 0 0.52149" rpy="${PI / 2} 0 0"/>
     <parent link="elbow_tilt_link"/>
@@ -222,5 +223,5 @@
     <dynamics damping="0.7"/>
   </joint>
-  <joint name="joint4" type="revolute">
+  <joint name="joint5" type="revolute">
     <origin xyz="-0.00038 0 0.0897" rpy="0 0 0"/>
     <parent link="wrist_tilt_link"/>
@@ -230,5 +231,5 @@
     <dynamics damping="0.7"/>
   </joint>
-  <joint name="l_gripper_joint" type="revolute">
+  <joint name="l_gripper_joint" type="fixed">
     <origin xyz="0.03865 0 0" rpy="0 ${-PI / 2} 0"/>
     <parent link="wrist_yaw_link"/>
@@ -237,5 +238,5 @@
     <limit lower="-0.4" upper="1" effort="30" velocity="1.0"/>
   </joint>
-  <joint name="r_gripper_joint" type="revolute">
+  <joint name="r_gripper_joint" type="fixed">
     <origin xyz="-0.03865 0 0" rpy="0 ${-PI / 2} -3.14159"/>
     <parent link="wrist_yaw_link"/>
@@ -244,5 +245,5 @@
     <limit lower="-0.4" upper="1" effort="30" velocity="1.0"/>
   </joint>
-  <joint name="l_inner_gripper_joint" type="revolute">
+  <joint name="l_inner_gripper_joint" type="fixed">
     <origin xyz="0.01065 0 0" rpy="0 ${-PI / 2} 0"/>
     <parent link="wrist_yaw_link"/>
@@ -252,5 +253,5 @@
     <mimic joint="l_gripper_joint" multiplier="-1" offset="0" />
   </joint>
-  <joint name="r_inner_gripper_joint" type="revolute">
+  <joint name="r_inner_gripper_joint" type="fixed">
     <origin xyz="-0.01065 0 0" rpy="0 ${-PI / 2} -3.14159"/>
     <parent link="wrist_yaw_link"/>
@@ -260,5 +261,5 @@
     <mimic joint="r_gripper_joint" multiplier="-1" offset="${pi}" />
   </joint>
-  <joint name="l_finger_joint" type="revolute">
+  <joint name="l_finger_joint" type="fixed">
     <origin xyz="${0.037 + 0.028} 0 0" rpy="0 ${PI / 2} 0"/>
     <parent link="l_gripper_outer_link"/>
@@ -268,5 +269,5 @@
     <mimic joint="l_gripper_joint" multiplier="-1" offset="0" />
   </joint>
-  <joint name="r_finger_joint" type="revolute">
+  <joint name="r_finger_joint" type="fixed">
     <origin xyz="${0.037 + 0.028} 0 0" rpy="0 ${PI / 2} 0"/>
     <parent link="r_gripper_outer_link"/>
@@ -276,21 +277,11 @@
     <limit lower="-3.14" upper="3.14" effort="30" velocity="1.0"/>
   </joint>
-    <transmission name="tran0">
-      <type>transmission_interface/SimpleTransmission</type>
-      <joint name="joint0">
-          <hardwareInterface>hardware_interface/PositionJointInterface</hardwareInterface>
-      </joint>
-      <actuator name="motor0">
-          <hardwareInterface>hardware_interface/PositionJointInterface</hardwareInterface>
-          <mechanicalReduction>1</mechanicalReduction>
-      </actuator>
-  </transmission>
   <transmission name="tran1">
       <type>transmission_interface/SimpleTransmission</type>
       <joint name="joint1">
-          <hardwareInterface>hardware_interface/PositionJointInterface</hardwareInterface>
+          <hardwareInterface>hardware_interface/EffortJointInterface</hardwareInterface>
       </joint>
       <actuator name="motor1">
-          <hardwareInterface>hardware_interface/PositionJointInterface</hardwareInterface>
+          <hardwareInterface>hardware_interface/EffortJointInterface</hardwareInterface>
           <mechanicalReduction>1</mechanicalReduction>
       </actuator>
@@ -299,8 +290,8 @@
       <type>transmission_interface/SimpleTransmission</type>
       <joint name="joint2">
-          <hardwareInterface>hardware_interface/PositionJointInterface</hardwareInterface>
+          <hardwareInterface>hardware_interface/EffortJointInterface</hardwareInterface>
       </joint>
       <actuator name="motor2">
-          <hardwareInterface>hardware_interface/PositionJointInterface</hardwareInterface>
+          <hardwareInterface>hardware_interface/EffortJointInterface</hardwareInterface>
           <mechanicalReduction>1</mechanicalReduction>
       </actuator>
@@ -309,8 +300,8 @@
       <type>transmission_interface/SimpleTransmission</type>
       <joint name="joint3">
-          <hardwareInterface>hardware_interface/PositionJointInterface</hardwareInterface>
+          <hardwareInterface>hardware_interface/EffortJointInterface</hardwareInterface>
       </joint>
       <actuator name="motor3">
-          <hardwareInterface>hardware_interface/PositionJointInterface</hardwareInterface>
+          <hardwareInterface>hardware_interface/EffortJointInterface</hardwareInterface>
           <mechanicalReduction>1</mechanicalReduction>
       </actuator>
@@ -319,8 +310,18 @@
       <type>transmission_interface/SimpleTransmission</type>
       <joint name="joint4">
-          <hardwareInterface>hardware_interface/PositionJointInterface</hardwareInterface>
+          <hardwareInterface>hardware_interface/EffortJointInterface</hardwareInterface>
       </joint>
       <actuator name="motor4">
-          <hardwareInterface>hardware_interface/PositionJointInterface</hardwareInterface>
+          <hardwareInterface>hardware_interface/EffortJointInterface</hardwareInterface>
+          <mechanicalReduction>1</mechanicalReduction>
+      </actuator>
+  </transmission>
+  <transmission name="tran5">
+      <type>transmission_interface/SimpleTransmission</type>
+      <joint name="joint5">
+          <hardwareInterface>hardware_interface/EffortJointInterface</hardwareInterface>
+      </joint>
+      <actuator name="motor5">
+          <hardwareInterface>hardware_interface/EffortJointInterface</hardwareInterface>
           <mechanicalReduction>1</mechanicalReduction>
       </actuator>
